File: hardware/anemometers/ultrasonic/pcb/u_anemometer.kicad_sch (KiCad schematic)
At the start: 0 parts

Commit message: DRC clear
Other:
- removed sheet 4_rain
Changed lines of the file:
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@@
 	(paper "A4")
-	(sheet
-		(at 25.4 68.58)
-		(size 12.7 3.81)
-		(exclude_from_sim no)
-		(in_bom yes)
-		(on_board yes)
-		(dnp no)
-		(fields_autoplaced yes)
-		(stroke
-			(width 0.1524)
-			(type solid)
-		)
-		(fill
-			(color 0 0 0 0.0000)
-		)
-		(property "Sheetname" "4_rain"
-			(at 25.4 67.8684 0)
-			(effects
-				(font
-					(size 1.27 1.27)
-				)
-				(justify left bottom)
-			)
-		)
-		(property "Sheetfile" "4_rain.kicad_sch"
-			(at 25.4 72.9746 0)
-			(effects
-				(font
-					(size 1.27 1.27)
-				)
-				(justify left top)
-			)
-		)
-		(instances
-			(project "ProDoc_1-PCB_PCB_2021-01-26_22-01-27_2026-01-16"
-				(path "/a30633bf-68dd-4888-88d6-d1ee9beba30f"
-					(page "5")
-				)
-			)
-		)
-	)
 	(sheet
 		(at 25.4 41.91)
@@
 		)
 		(instances
-			(project "ProDoc_1-PCB_PCB_2021-01-26_22-01-27_2026-01-16"
+			(project "u_anemometer"
 				(path "/a30633bf-68dd-4888-88d6-d1ee9beba30f"
 					(page "3")
@@
 		)
 		(instances
-			(project "ProDoc_1-PCB_PCB_2021-01-26_22-01-27_2026-01-16"
+			(project "u_anemometer"
 				(path "/a30633bf-68dd-4888-88d6-d1ee9beba30f"
 					(page "2")
@@
 		)
 		(instances
-			(project "ProDoc_1-PCB_PCB_2021-01-26_22-01-27_2026-01-16"
+			(project "u_anemometer"
 				(path "/a30633bf-68dd-4888-88d6-d1ee9beba30f"
 					(page "4")
