File: hardware/anemometers/ultrasonic/pcb/u_anemometer.kicad_pcb (KiCad board)
At the start: 4 copper layers, 46 x 46 mm, 162 parts

Commit message: update
Parts:
- renumbered CAN to CAN1, DEBUG to DEBUG1, EAST to EAST1, I2C to I2C1, NORTH to NORTH1, SOUTH to SOUTH1, SPI to SPI1, USB to USB1, WEST to WEST1

Commit message: Updaetes
Parts:
- removed ANT: , ProDoc_1-PCB_PCB_2021-01-26_22-01-27_2026-01-16:INDUCTOR_COILCRAFT_MA5532-AE
- removed C54, C56: , ProDoc_1-PCB_PCB_2021-01-26_22-01-27_2026-01-16:C0402
- removed C55: , ProDoc_1-PCB_PCB_2021-01-26_22-01-27_2026-01-16:C0603
- removed IR1: , ProDoc_1-PCB_PCB_2021-01-26_22-01-27_2026-01-16:LED-TH_BD3.0-P2.54-FD
- removed IRR: , ProDoc_1-PCB_PCB_2021-01-26_22-01-27_2026-01-16:LED-TH_BD3.1-P2.54-FD
- removed MIC1: , ProDoc_1-PCB_PCB_2021-01-26_22-01-27_2026-01-16:MIC-SMD_5P-L3.0-W4.0-P0.85-BL
- removed R42, R45: , ProDoc_1-PCB_PCB_2021-01-26_22-01-27_2026-01-16:R0402
- removed R43: , ProDoc_1-PCB_PCB_2021-01-26_22-01-27_2026-01-16:R0603
- removed U11: , ProDoc_1-PCB_PCB_2021-01-26_22-01-27_2026-01-16:16LDMLPQ
- BAT1: renamed from BAT; value (none) -> B2B-XH-A-GU
- C1, C13, C2, C22, C24, C32, C34, C44: value (none) -> 1uF
- C12: value (none) -> 100uF
- C14, C16, C36, C4, C45: value (none) -> 4.7uF
- C15, C23, C9: value (none) -> 10nF
- C17, C18, C19, C21, C26, C31, C33, C35, C40, C46, C47, C50, C51, C52, C8: value (none) -> 100nF
- C25, C27, C28, C29, C30, C37, C38, C41, C42, C43: value (none) -> 2.2uF
- C3, C5, C6, C7: value (none) -> 10pF
- C39: value (none) -> 22pF
- CAN1, I2C1, UART1, UART2: value (none) -> 1.25T-1-4A
- D1: value (none) -> NUP1105LT1G
- D10, D11, D12, D13, D14, D15, D16, D17, D18, D19, D4, D5, D6, D7, D8, D9: value (none) -> 1N4148WS T4
- D2: value (none) -> SN65220DBVR
- D3: value (none) -> B5819W_C8598
- DEBUG1: value (none) -> 2328702-8
- EAST1, NORTH1, SOUTH1, WEST1: value (none) -> 1.25T-2P-DP
- LED1: value (none) -> 19-217/BHC-ZL1M2RY/3T
- LED2: value (none) -> KT-0603R
- Q1, Q2: value (none) -> SI2301CDS-T1-GE3
- R1: value (none) -> 120
- R10: value (none) -> 0
- R11, R15, R25, R3, R30, R34, R35, R39, R8, R9: value (none) -> 100K
- R12, R16, R21, R26, R31, R32, R33, R36, R40: value (none) -> 4.7K
- R13, R14, R17, R18, R19, R2, R20, R22, R23, R27, R28, R29, R37, R38, R41: value (none) -> 10K
- R24, R4, R5: value (none) -> 33
- R6, R7: value (none) -> 1K
- RST1: renamed from RST; value (none) -> B3U-1000P
- SD1: renamed from SD; value (none) -> SDCARD MOLEX 1040310811
- SPI1: value (none) -> 1.25T-8A_C722648
- SW1: value (none) -> B3U-1000P
- SWD1: renamed from SWD; value (none) -> 4pad
- U1: value (none) -> TCAN330GDCNR
- U2: value (none) -> STM32L476RGT6
- U3: value (none) -> XC6206P332MR
- U4, U6: value (none) -> MAX3222EIPWR
- U5: value (none) -> SN74LV4052APW
- U7: value (none) -> LMV358B-VR
- U8: value (none) -> BME280
- U9: value (none) -> BMX160
- UART3: renamed from UART; value (none) -> 4pad
- USB1: value (none) -> 47346-0001
- X1: value (none) -> 32.768KHz
- X2: value (none) -> 25M
Connections:
- net ADC_CH3 renamed /1_mcu/ADC_CH3
- net BAT_2 renamed Net-(D3-+)
- net C24_2 renamed Net-(U6-DOUT2)
- net C32_2 renamed Net-(U4-DOUT1)
- net C33_2 renamed Net-(D10-K)
- net C34_2 renamed Net-(U4-DOUT2)
- net C37_1 renamed Net-(U6-C1+)
- net C37_2 renamed Net-(U6-C1−)
- net C41_1 renamed Net-(U6-V+)
- net C42_1 renamed Net-(U6-C2+)
- net C42_2 renamed Net-(U6-C2−)
- net C43_2 renamed Net-(U6-V−)
- net C44_2 renamed Net-(U6-DOUT1)
- net CAN_RX renamed /1_mcu/CAN_RX
- net CAN_TX renamed /1_mcu/CAN_TX
- net D12_1 renamed Net-(D12-K)
- net D12_2 renamed Net-(D12-A)
- net D16_1 renamed Net-(D16-K)
- net D16_2 renamed Net-(D16-A)
- net D2_1 renamed Net-(USB1-Data-)
- net D2_3 renamed Net-(USB1-Data+)
- net D4_1 renamed Net-(D4-K)
- net D4_2 renamed Net-(D4-A)
- net D9_1 renamed Net-(D8-A)
- net EAST_IN renamed /2_anemometer/EAST_IN
- net EAST_OUT renamed /2_anemometer/EAST_OUT
- net LED1_1 renamed Net-(LED1-A)
- net NORTH_IN renamed /2_anemometer/NORTH_IN
- net NORTH_OUT renamed /2_anemometer/NORTH_OUT
- net Q2_1 renamed Net-(Q2-G)
- net R12_2 renamed Net-(D6-K)
- net R21_1 renamed Net-(D8-K)
- net R26_2 renamed Net-(D14-K)
- net R36_2 renamed Net-(D18-K)
- net R7_1 renamed Net-(LED2-A)
- net RST renamed /1_mcu/RST
- net SDMMC1_CK renamed /1_mcu/SDMMC1_CK
- net SDMMC1_CMD renamed /1_mcu/SDMMC1_CMD
- net SDMMC1_D0 renamed /1_mcu/SDMMC1_D0
- net SDMMC1_D1 renamed /1_mcu/SDMMC1_D1
- net SDMMC1_D2 renamed /1_mcu/SDMMC1_D2
- net SDMMC1_D3 renamed /1_mcu/SDMMC1_D3
- net SD_4 renamed Net-(Q1-D)
- net SOUTH_IN renamed /2_anemometer/SOUTH_IN
- net SOUTH_OUT renamed /2_anemometer/SOUTH_OUT
- net SPI1_CS0 renamed /1_mcu/SPI1_CS0
- net SPI1_CS1 renamed /1_mcu/SPI1_CS1
- net SPI1_MISO renamed /1_mcu/SPI1_MISO
- net SPI1_MOSI renamed /1_mcu/SPI1_MOSI
- net SPI1_SCK renamed /1_mcu/SPI1_SCK
- net SWCLK renamed /1_mcu/SWCLK
- net SWDIO renamed /1_mcu/SWDIO
- net TIM3_CH1 renamed PWM_IN
- net U1_6 renamed Net-(U1-CANL)
- net U1_7 renamed Net-(U1-CANH)
- net U2_2 renamed Net-(U1-S)
- net U2_3 renamed Net-(U2-PC14/OSC32_IN)
- net U2_36 renamed Net-(U2-PB15)
- net U2_37 renamed Net-(U2-PC6)
- net U2_38 renamed Net-(U2-PC7)
- net U2_4 renamed Net-(U2-PC15/OSC32_OUT)
- net U2_43 renamed Net-(SD1-SH3)
- net U2_5 renamed Net-(U2-PH0/OSCIN)
- net U2_50 renamed Net-(Q1-G)
- net U2_6 renamed Net-(U2-PH1/OSCOUT)
- net U2_60 renamed Net-(U2-BOOT0)
- net U4_2 renamed Net-(U4-C1+)
- net U4_3 renamed Net-(U4-V+)
- net U4_4 renamed Net-(U4-C1−)
- net U4_5 renamed Net-(U4-C2+)
- net U4_6 renamed Net-(U4-C2−)
- net U4_7 renamed Net-(U4-V−)
- net U5_3 renamed Net-(U5-Y)
- net U7_2 renamed Net-(U7A-INA-)
- net U7_3 renamed Net-(U7A-INA+)
- net U7_5 renamed Net-(U7B-INB+)
- net U7_6 renamed Net-(U7B-INB-)
- net USART1_RX renamed /1_mcu/USART1_RX
- net USART1_TX renamed /1_mcu/USART1_TX
- net USART2_RX renamed /1_mcu/USART2_RX
- net USART2_TX renamed /1_mcu/USART2_TX
- net USART3_RX renamed /1_mcu/USART3_RX
- net USART3_TX renamed /1_mcu/USART3_TX
- net USB_DM renamed /1_mcu/USB_DM
- net USB_DP renamed /1_mcu/USB_DP
- net WEST_IN renamed /2_anemometer/WEST_IN
- net WEST_OUT renamed /2_anemometer/WEST_OUT
- D2 pad 5: D2_5 -> unconnected-(D2-Pad5)
- DEBUG1 pad 5: DEBUG_5 -> unconnected-(DEBUG1-Pad5)
- R29 pad 1: U7_1 -> Net-(U7A-OUTA)
- R31 pad 2: U7_1 -> Net-(U7A-OUTA)
- SPI1 pad 7: SPI_7 -> unconnected-(SPI1-Pad7)
- U2 pad 10: MIC_CLK -> unconnected-(U2-PC2-Pad10)
- U2 pad 15: RAIN_SENS -> unconnected-(U2-PA1-Pad15)
- U2 pad 20: RAIN_LED -> unconnected-(U2-PA4-Pad20)
- U2 pad 41: U2_41 -> unconnected-(U2-PA8-Pad41)
- U2 pad 42: U2_42 -> unconnected-(U2-PA9-Pad42)
- U2 pad 8: MIC_DAT -> unconnected-(U2-PC0-Pad8)
- U2 pad 9: U2_9 -> unconnected-(U2-PC1-Pad9)
- U4 pad 10: U4_10 -> unconnected-(U4-ROUT2-Pad10)
- U4 pad 11: U4_11 -> unconnected-(U4-NC-Pad11)
- U4 pad 14: U4_14 -> unconnected-(U4-NC-Pad14)
- U4 pad 15: U4_15 -> unconnected-(U4-ROUT1-Pad15)
- U4 pad 16: U4_16 -> unconnected-(U4-RIN1-Pad16)
- U4 pad 9: U4_9 -> unconnected-(U4-RIN2-Pad9)
- U6 pad 10: U6_10 -> unconnected-(U6-ROUT2-Pad10)
- U6 pad 11: U6_11 -> unconnected-(U6-NC-Pad11)
- U6 pad 14: U6_14 -> unconnected-(U6-NC-Pad14)
- U6 pad 15: U6_15 -> unconnected-(U6-ROUT1-Pad15)
- U6 pad 16: U6_16 -> unconnected-(U6-RIN1-Pad16)
- U6 pad 9: U6_9 -> unconnected-(U6-RIN2-Pad9)
- U7 pad 1: U7_1 -> Net-(U7A-OUTA)
- U9 pad 10: U9_10 -> unconnected-(U9-OCSB-Pad10)
- U9 pad 11: U9_11 -> unconnected-(U9-OSDO-Pad11)
- U9 pad 4: U9_4 -> unconnected-(U9-INT1-Pad4)
- U9 pad 9: U9_9 -> unconnected-(U9-INT2-Pad9)
- USB1 pad 4: USB_4 -> unconnected-(USB1-ID-Pad4)
Routing:
- net SCL: track 85.1 -> 55.8 mm, vias 3 -> 1
- net SDA: track 87.4 -> 59.1 mm, vias 7 -> 5
- net GND: track 265.6 -> 241.2 mm, vias 120 -> 115
- net AS3935_INT: track 18.5 -> 0.00 mm, vias 2 -> 0
- net RAIN_LED: track 13.8 -> 0.00 mm, vias 1 -> 0
- net 3.3V: track 104.3 -> 92.7 mm, vias 21 -> 18
- net U11_3: track 10.9 -> 0.00 mm, vias 1 -> 0
- net RAIN_SENS: track 13.7 -> 5.13 mm, vias 1 -> 0
- net MIC_CLK: track 5.34 -> 0.00 mm
- net R43_1: track 4.68 -> 0.00 mm
- net MIC_DAT: track 4.13 -> 0.00 mm
- net U11_1: track 3.36 -> 0.00 mm
- net IR1_2: track 3.20 -> 0.00 mm
- net unconnected-(U2-PA1-Pad15): track 0.00 -> 2.38 mm

Commit message: Latest updates!
Other:
- board text removed: "2021/02/28"
- board text removed: "By Jianjia Ma"
- board text removed: "QingStation"
- board text removed: "Ver1.1"

Commit message: Update to BMI270
Connections:
- ? pad 2: U7_1 -> Net-(U7A-OUTA)
Routing:
- net U7_1: track 5.00 -> 0.00 mm, vias 1 -> 0
- net Net-(U7A-OUTA): track 0.00 -> 5.00 mm, vias 0 -> 1
Changed lines of the file:
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@@
 	(net 133 "R43_1")
 	(net 134 "Q3_1")
-	(net 135 "U7_1")
-	(net 136 "U10_5")
-	(net 137 "U10_4")
+	(net 135 "U10_5")
+	(net 136 "U10_4")
 	(footprint "ProDoc_1-PCB_PCB_2021-01-26_22-01-27_2026-01-16:C0402"
 		(layer "F.Cu")
@@
 			(size 2 2)
 			(layers "B.Cu" "B.Mask" "B.Paste")
-			(net 135 "U7_1")
+			(net 80 "Net-(U7A-OUTA)")
 			(thermal_bridge_angle 90)
 		)
@@
 			(size 0.95 0.4)
 			(layers "B.Cu" "B.Mask" "B.Paste")
-			(net 137 "U10_4")
+			(net 136 "U10_4")
 		)
 		(pad "5" smd rect
@@
 			(size 0.95 0.4)
 			(layers "B.Cu" "B.Mask" "B.Paste")
-			(net 136 "U10_5")
+			(net 135 "U10_5")
 		)
 		(pad "6" smd rect
@@
 	)
 	(segment
+		(start 142.2505 127.6505)
+		(end 141.4505 128.4505)
+		(width 0.2)
+		(layer "F.Cu")
+		(net 80)
+	)
+	(segment
+		(start 142.9745 127.0255)
+		(end 141.402 127.0255)
+		(width 0.2)
+		(layer "F.Cu")
+		(net 80)
+	)
+	(segment
+		(start 142.2505 127.0255)
+		(end 142.2505 127.6505)
+		(width 0.2)
+		(layer "F.Cu")
+		(net 80)
+	)
+	(segment
+		(start 141.4505 128.4505)
+		(end 140.099 128.4505)
+		(width 0.2)
+		(layer "F.Cu")
+		(net 80)
+	)
+	(segment
+		(start 143.2005 126.7995)
+		(end 142.9745 127.0255)
+		(width 0.2)
+		(layer "F.Cu")
+		(net 80)
+	)
+	(via
+		(at 141.4505 128.4505)
+		(size 0.6095)
+		(drill 0.305)
+		(layers "F.Cu" "B.Cu")
+		(net 80)
+	)
+	(segment
 		(start 142.4995 125.4)
 		(end 142.1745 125.725)
@@
 		(net 134)
 	)
-	(segment
-		(start 142.2505 127.6505)
-		(end 141.4505 128.4505)
-		(width 0.2)
-		(layer "F.Cu")
-		(net 135)
-	)
-	(segment
-		(start 142.9745 127.0255)
-		(end 141.402 127.0255)
-		(width 0.2)
-		(layer "F.Cu")
-		(net 135)
-	)
-	(segment
-		(start 142.2505 127.0255)
-		(end 142.2505 127.6505)
-		(width 0.2)
-		(layer "F.Cu")
-		(net 135)
-	)
-	(segment
-		(start 141.4505 128.4505)
-		(end 140.099 128.4505)
-		(width 0.2)
-		(layer "F.Cu")
-		(net 135)
-	)
-	(segment
-		(start 143.2005 126.7995)
-		(end 142.9745 127.0255)
-		(width 0.2)
-		(layer "F.Cu")
-		(net 135)
-	)
-	(via
-		(at 141.4505 128.4505)
-		(size 0.6095)
-		(drill 0.305)
-		(layers "F.Cu" "B.Cu")
-		(net 135)
-	)
 	(zone

Commit message: Fab outputs
Parts:
- added REF**: MountingHole_2.2mm_M2_ISO14580, MountingHole:MountingHole_2.2mm_M2_ISO14580, F.Cu at (168.2, 121.7)
- added REF**: MountingHole_2.2mm_M2_ISO14580, MountingHole:MountingHole_2.2mm_M2_ISO14580, F.Cu at (157.3, 128.1)
- added REF**: MountingHole_2.2mm_M2_ISO14580, MountingHole:MountingHole_2.2mm_M2_ISO14580, F.Cu at (138.8, 110.1)
- moved ? 2.06 mm to (139.9, 113.1)
Routing:
- net ECHO_OUT: track 32.3 -> 31.7 mm
- net GND: track 241.2 -> 241.0 mm, vias 115 -> 114

Commit message: Fixed!
Parts:
- renumbered VBAT to VBAT1
Changed lines of the file:
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@@
 		(layer "F.Cu")
 		(at 140.25 104.15 -90)
-		(property "Reference" "VBAT"
-			(at -1.8 1.85 270)
+		(property "Reference" "VBAT1"
+			(at -1.8 1.85 90)
 			(layer "F.SilkS")
 			(hide yes)
@@
 				(font
 					(size 0.48 0.44)
-					(thickness 0.1525)
+					(thickness 0.11)
 				)
-				(justify left bottom)
+				(justify right top)
 			)
 		)
 		(property "Value" ""
-			(at 0 0 270)
+			(at 0 0 90)
 			(layer "F.Fab")
 			(effects
@@
 		)
 		(property "Datasheet" ""
-			(at 0 0 270)
+			(at 0 0 90)
 			(layer "F.Fab")
 			(hide yes)
@@
 		)
 		(property "Description" ""
-			(at 0 0 270)
+			(at 0 0 90)
 			(layer "F.Fab")
 			(hide yes)
@@
 		)
 		(property "JLC_3DModel_Q" "624118aa3cc7497086c383c2d72e0852"
-			(at 0 0 270)
+			(at 0 0 90)
 			(layer "Cmts.User")
 			(hide yes)
@@
 		)
 		(property "JLC_3D_Size" "1.6 0.8"
-			(at 0 0 270)
+			(at 0 0 90)
 			(layer "Cmts.User")
 			(hide yes)
